Commit message: starting my_tape_follower shaya

File: src/robot_car/src/description/robot_car_description.urdf (robot description, URDF)
Before this commit: robot robot_car, 0 links, 0 joints
Links:
- added link base_footprint
- added link base_link; collision box size=${base_length} ${base_width} ${base_height}; visual box size=${base_length} ${base_width} ${base_height}
- added link camera_link, mass 0.035; collision box size=0.015 0.130 0.022; visual box size=0.015 0.130 0.022
- added link front_caster; collision sphere radius=${(wheel_radius+wheel_zoff-(base_height/2))}; visual sphere radius=${(wheel_radius+wheel_zoff-(base_height/2))}
- added link imu_link; collision box size=0.1 0.1 0.1; visual box size=0.1 0.1 0.1
- added link lidar_link, mass 0.125; collision cylinder length=0.055 radius=0.0508; visual cylinder length=0.055 radius=0.0508
Joints:
- added joint base_joint: type fixed, parent base_link, child base_footprint, origin xyz=0.0 0.0 ${-(wheel_radius+wheel_zoff)} rpy=0 0 0
- added joint camera_joint: type fixed, parent base_link, child camera_link, origin xyz=0.215 0 0.05 rpy=0 0 0
- added joint caster_joint: type fixed, parent base_link, child front_caster, origin xyz=${caster_xoff} 0.0 ${-(base_height/2)} rpy=0 0 0
- added joint imu_joint: type fixed, parent base_link, child imu_link, origin xyz=0 0 0.01
- added joint lidar_joint: type fixed, parent base_link, child lidar_link, origin xyz=0 0 0.12 rpy=0 0 0
